File: 10A-Bias-T.kicad_pcb (KiCad board)
At the start: 2 copper layers, 181 x 62 mm, 60 parts, among them J1 Conn_Coaxial, J2 Conn_01x02_Female, J3 Conn_Coaxial, J4 Conn_Coaxial, J5 Conn_01x02_Female, J6 Conn_Coaxial

Commit message: Add files via upload
updated
Parts:
- added C3: 0.022µF, Capacitor_THT:C_Disc_D7.5mm_W5.0mm_P10.00mm, F.Cu at (36.0, 66.0)
- added C7: 0.022µF, Capacitor_THT:C_Disc_D7.5mm_W5.0mm_P10.00mm, F.Cu at (124.5, 68.5)
- added C8: 0.022µF, Capacitor_THT:C_Disc_D7.5mm_W5.0mm_P10.00mm, F.Cu at (118.0, 68.5)
- added C9: 0.022µF, Capacitor_THT:C_Disc_D7.5mm_W5.0mm_P10.00mm, F.Cu at (130.0, 68.5)
- C1, C2: value 33 pF -> 0.022µF; footprint Capacitor_THT:C_Disc_D8.0mm_W5.0mm_P7.50mm -> Capacitor_THT:C_Disc_D7.5mm_W5.0mm_P10.00mm
- moved C1 100.0 mm to (24.5, 66.0)
- moved C2 1.00 mm to (30.5, 66.0)
Connections:
- C1 pad 1: /RF2 -> /RF+DC
- C1 pad 2: /RF+DC2 -> /RF
Routing:
- net Earth: track 52.5 -> 205.5 mm
- net GND: track 42.3 -> 112.5 mm
- net /RF2: track 26.5 -> 36.0 mm
- net /RF: track 19.0 -> 28.0 mm
- net /RF+DC2: track 36.1 -> 42.6 mm
- net /RF+DC: track 38.5 -> 44.5 mm
Other:
- rule pad_to_mask_clearance: 0.05 -> 0
